File: kicadFiles/Dofleini-controller-STM32.sch (KiCad schematic (older format))
At the start: 32 parts, among them J1 Conn_ARM_JTAG_SWD_10, J2 Conn_01x09_Male, J3 TYPE-C-31-M12_13, J4 Conn_01x22_Male, J5 Conn_01x07_Male, Q1 DTC123J, Q2 AO4406AL, U1 STM32F072CBTx, U2 TLV1117-33, U3 USBLC6-2SC6

Commit message: Added mounting holes
Parts:
- added H1, H2: MountingHole, MountingHole:MountingHole_3.2mm_M3_ISO7380, symbol Mechanical:MountingHole
Changed lines of the file:
@@
 Wire Wire Line
 	3450 4250 3650 4250
+$Comp
+L Mechanical:MountingHole H2
+U 1 1 5E5268FD
+P 6300 1100
+F 0 "H2" H 6400 1146 50  0000 L CNN
+F 1 "MountingHole" H 6400 1055 50  0000 L CNN
+F 2 "MountingHole:MountingHole_3.2mm_M3_ISO7380" H 6300 1100 50  0001 C CNN
+F 3 "~" H 6300 1100 50  0001 C CNN
+	1    6300 1100
+	1    0    0    -1
+$EndComp
+$Comp
+L Mechanical:MountingHole H1
+U 1 1 5E526EE0
+P 6000 1100
+F 0 "H1" H 6100 1146 50  0000 L CNN
+F 1 "MountingHole" H 6100 1055 50  0000 L CNN
+F 2 "MountingHole:MountingHole_3.2mm_M3_ISO7380" H 6000 1100 50  0001 C CNN
+F 3 "~" H 6000 1100 50  0001 C CNN
+	1    6000 1100
+	1    0    0    -1
+$EndComp
 $EndSCHEMATC

Commit message: Added BOM
Parts:
- D1: value RBD60M-60TR -> RB060M-60TR
Changed lines of the file:
@@
 P 8100 3650
 F 0 "D1" V 8100 3450 50  0000 L CNN
-F 1 "RBD60M-60TR" V 8200 3050 50  0000 L CNN
+F 1 "RB060M-60TR" V 8200 3050 50  0000 L CNN
 F 2 "acheronComponents:D_SOD-123" V 8100 3650 50  0001 C CNN
 F 3 "~" V 8100 3650 50  0001 C CNN
